File: Schematics/KiCAD/FT8_Transceiver.kicad_sch (KiCad schematic)
At the start: 0 parts

Commit message: schematic
Parts:
- added U1: ~, ATS20+, symbol DL1SKD:ATS20+
- added U2: TXB0108DQSR, Package_SON:USON-20_2x4mm_P0.4mm, symbol Logic_LevelTranslator:TXB0108DQSR
Connections:
- new net: U1. (TX), U2.1 (A1)
- new net: U1. (TX), U2.15 (GND)
- new net: U1. (TX), U2.2 (A2)
- new net: U1. (TX), U2.5 (VCCA)
