File: ATS_EX_FT8_TX/Circuit/KiCad/TX_Modul/TX_Modul.kicad_sch (KiCad schematic)
At the start: 22 parts, among them J1 Conn_01x15_Socket, J2 Conn_01x15_Socket, J3 From PC, J4 Relais, J6 Conn_01x06_Socket, J7 Conn_01x06_Socket, J8 Conn_01x06_Socket

Commit message: LEDs added
Parts:
- added J9: StatusLED, Connector_PinSocket_2.54mm:PinSocket_1x03_P2.54mm_Vertical, symbol Connector:Conn_01x03_Socket
Connections:
- net at J2.7 (Pin_7), J4.3 (Pin_3): now also J2.12 (Pin_12), J9.1 (Pin_1)
- net at C2.1 (+), J2.10 (Pin_10), J2.4 (Pin_4)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: now also J9.2 (Pin_2)
- net at J2.8 (Pin_8): now also J9.3 (Pin_3)
Other:
- note added: "RX LED"
- note added: "TX LED"
Changed lines of the file:
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@@
 		)
 	)
+	(text "RX LED"
+		(exclude_from_sim no)
+		(at 159.258 45.466 0)
+		(effects
+			(font
+				(size 0.762 0.762)
+			)
+		)
+	)
 	(text "Levelshifter"
 		(exclude_from_sim no)
@@
 		)
 	)
+	(text "TX LED"
+		(exclude_from_sim no)
+		(at 158.75 55.626 0)
+		(effects
+			(font
+				(size 0.762 0.762)
+			)
+		)
+	)
 	(text "RX\n"
 		(exclude_from_sim no)
@@
 	)
 	(junction
+		(at 184.15 66.04)
+		(diameter 0)
+		(color 0 0 0 0)
+	)
+	(junction
 		(at 78.74 71.12)
 		(diameter 0)
@@
 	)
 	(junction
+		(at 184.15 58.42)
+		(diameter 0)
+		(color 0 0 0 0)
+	)
+	(junction
 		(at 201.93 92.71)
 		(diameter 0)
@@
 		(color 0 0 0 0)
 	)
+	(junction
+		(at 176.53 68.58)
+		(diameter 0)
+		(color 0 0 0 0)
+	)
+	(wire
+		(pts
+			(xy 184.15 58.42) (xy 184.15 66.04)
+		)
+		(stroke
+			(width 0)
+			(type default)
+		)
+	)
 	(wire
 		(pts
@@
 	(wire
 		(pts
-			(xy 184.15 115.57) (xy 184.15 58.42)
+			(xy 132.08 58.42) (xy 73.66 58.42)
 		)
 		(stroke
@@
 	(wire
 		(pts
-			(xy 132.08 58.42) (xy 73.66 58.42)
+			(xy 132.08 40.64) (xy 106.68 40.64)
 		)
 		(stroke
@@
 	(wire
 		(pts
-			(xy 132.08 40.64) (xy 106.68 40.64)
+			(xy 76.2 113.03) (xy 76.2 92.71)
 		)
 		(stroke
@@
 	(wire
 		(pts
-			(xy 76.2 113.03) (xy 76.2 92.71)
+			(xy 55.88 46.99) (xy 55.88 71.12)
 		)
 		(stroke
@@
 	(wire
 		(pts
-			(xy 55.88 46.99) (xy 55.88 71.12)
+			(xy 50.8 44.45) (xy 59.69 44.45)
 		)
 		(stroke
@@
 	(wire
 		(pts
-			(xy 50.8 44.45) (xy 59.69 44.45)
+			(xy 168.91 71.12) (xy 168.91 55.88)
+		)
+		(stroke
+			(width 0)
+			(type default)
+		)
+	)
+	(wire
+		(pts
+			(xy 184.15 45.72) (xy 184.15 58.42)
 		)
 		(stroke
@@
 	(wire
 		(pts
-			(xy 176.53 66.04) (xy 176.53 113.03)
+			(xy 176.53 66.04) (xy 176.53 68.58)
 		)
 		(stroke
@@
 	(wire
 		(pts
+			(xy 184.15 66.04) (xy 184.15 115.57)
+		)
+		(stroke
+			(width 0)
+			(type default)
+		)
+	)
+	(wire
+		(pts
 			(xy 25.4 49.53) (xy 33.02 49.53)
 		)
@@
 	(wire
 		(pts
+			(xy 168.91 55.88) (xy 154.94 55.88)
+		)
+		(stroke
+			(width 0)
+			(type default)
+		)
+	)
+	(wire
+		(pts
+			(xy 200.66 66.04) (xy 184.15 66.04)
+		)
+		(stroke
+			(width 0)
+			(type default)
+		)
+	)
+	(wire
+		(pts
 			(xy 106.68 113.03) (xy 120.65 113.03)
 		)
@@
 	(wire
 		(pts
+			(xy 154.94 45.72) (xy 184.15 45.72)
+		)
+		(stroke
+			(width 0)
+			(type default)
+		)
+	)
+	(wire
+		(pts
 			(xy 81.28 73.66) (xy 81.28 50.8)
 		)
@@
 	(wire
 		(pts
+			(xy 200.66 71.12) (xy 168.91 71.12)
+		)
+		(stroke
+			(width 0)
+			(type default)
+		)
+	)
+	(wire
+		(pts
 			(xy 106.68 105.41) (xy 106.68 113.03)
 		)
@@
 	(wire
 		(pts
+			(xy 176.53 68.58) (xy 200.66 68.58)
+		)
+		(stroke
+			(width 0)
+			(type default)
+		)
+	)
+	(wire
+		(pts
 			(xy 180.34 97.79) (xy 201.93 97.79)
 		)
@@
 	(wire
 		(pts
+			(xy 176.53 68.58) (xy 176.53 113.03)
+		)
+		(stroke
+			(width 0)
+			(type default)
+		)
+	)
+	(wire
+		(pts
 			(xy 54.61 73.66) (xy 81.28 73.66)
 		)
@@
 					(unit 1)
 				)
+			)
+		)
+	)
+	(symbol
+		(lib_id "Connector:Conn_01x03_Socket")
+		(at 205.74 68.58 0)
+		(unit 1)
+		(body_style 1)
+		(exclude_from_sim no)
+		(in_bom yes)
+		(on_board yes)
+		(in_pos_files yes)
+		(dnp no)
+		(property "Reference" "J9"
+			(at 203.962 60.198 0)
+			(show_name no)
+			(do_not_autoplace no)
+			(effects
+				(font
+					(size 1.27 1.27)
+				)
+				(justify left)
+			)
+		)
+		(property "Value" "StatusLED"
+			(at 203.708 62.738 0)
+			(show_name no)
+			(do_not_autoplace no)
+			(effects
+				(font
+					(size 1.27 1.27)
+				)
+				(justify left)
+			)
+		)
+		(property "Footprint" "Connector_PinSocket_2.54mm:PinSocket_1x03_P2.54mm_Vertical"
+			(at 205.74 68.58 0)
+			(hide yes)
+			(show_name no)
+			(do_not_autoplace no)
+			(effects
+				(font
+					(size 1.27 1.27)
+				)
+			)
+		)
+		(property "Datasheet" ""
+			(at 205.74 68.58 0)
+			(hide yes)
+			(show_name no)
+			(do_not_autoplace no)
+			(effects
+				(font
+					(size 1.27 1.27)
+				)
+			)
+		)
+		(property "Description" "Generic connector, single row, 01x03, script generated"
+			(at 205.74 68.58 0)
+			(hide yes)
+			(show_name no)
+			(do_not_autoplace no)
+			(effects
+				(font
+					(size 1.27 1.27)
+				)
+			)
+		)
+		(pin "1"
+		)
+		(pin "2"
+		)
+		(pin "3"
+		)
+		(instances
+			(project "TX_Modul"
+				(path "/a9cb15dd-917f-4e9c-8fab-e72d6e2fbc01"
+					(reference "J9")
+					(unit 1)
+				)
